File: PCB/Base_Arduino.sch (KiCad schematic (older format))
At the start: 15 parts, among them IC1 ATMEGA328-P, X1 CRYSTAL

Commit message: Libraries and footprints adjustments. New connectors (4 pins main, 2 pins debug and 6 pins isp). New source input cap.
Parts:
- added C10: 100nF, Capacitors_ThroughHole:C_Rect_L7_W2.5_P5, symbol C
- C5, C6: footprint ArduBooster_Library:CAP_SMALL -> Capacitors_ThroughHole:C_Rect_L7_W2_P5; symbol C-RESCUE-ArduBooster -> C
- C7: footprint ArduBooster_Library:CAP_BIG -> Capacitors_ThroughHole:C_Rect_L7_W4.5_P5; symbol C-RESCUE-ArduBooster -> C
- C8, C9: footprint ArduBooster_Library:CAP_MID -> Capacitors_ThroughHole:C_Rect_L7_W2.5_P5; symbol C-RESCUE-ArduBooster -> C
- IC1: symbol ATMEGA328-P-RESCUE-ArduBooster -> ATMEGA328-P
- R2, R3, R4, R5, R6, R7, R8, R9: symbol R-RESCUE-ArduBooster -> R
- X1: symbol CRYSTAL -> Crystal
Connections:
- net +5V: now also C10.1
- net GNDREF: now also C10.2
Changed lines of the file:
@@
 EESchema Schematic File Version 2
-LIBS:ArduBooster-rescue
 LIBS:power
 LIBS:device
@@
 Rev "1.0"
 Comp ""
-Comment1 ""
+Comment1 "Basic Arduino setup"
 Comment2 ""
 Comment3 ""
@@
 $EndDescr
 $Comp
-L ATMEGA328-P-RESCUE-ArduBooster IC1
+L ATMEGA328-P IC1
 U 1 1 54D7F099
 P 3600 3750
 F 0 "IC1" H 2850 5000 40  0000 L BNN
 F 1 "ATMEGA328-P" H 4000 2350 40  0000 L BNN
-F 2 "Sockets_DIP:DIP-28__300" H 3600 3750 30  0000 C CIN
+F 2 "Sockets_DIP:DIP-28__300" H 3600 3750 30  0001 C CIN
 F 3 "" H 3600 3750 60  0000 C CNN
 	1    3600 3750
@@
 $EndComp
 $Comp
-L CRYSTAL X1
+L Crystal X1
 U 1 1 54D7F8BC
 P 6500 3300
@@
 	6250 3350 6250 3650
 Wire Wire Line
-	6250 3650 6750 3650
-Wire Wire Line
-	6500 3650 6500 3600
+	6250 3650 6800 3650
+Wire Wire Line
+	6500 3450 6500 3650
 Wire Wire Line
 	4600 3250 6250 3250
@@
 	6250 3250 6250 2950
 Wire Wire Line
-	6250 2950 6750 2950
-Wire Wire Line
-	6500 2950 6500 3000
-$Comp
-L C-RESCUE-ArduBooster C5
+	6250 2950 6800 2950
+Wire Wire Line
+	6500 2950 6500 3150
+$Comp
+L C C5
 U 1 1 54D7FA47
 P 6950 2950
 F 0 "C5" H 7000 3050 50  0000 L CNN
 F 1 "22p" H 7000 2850 50  0000 L CNN
-F 2 "ArduBooster_Library:CAP_SMALL" H 6988 2800 30  0001 C CNN
+F 2 "Capacitors_ThroughHole:C_Rect_L7_W2_P5" H 6988 2800 30  0001 C CNN
 F 3 "" H 6950 2950 60  0000 C CNN
 	1    6950 2950
@@
 $EndComp
 $Comp
-L C-RESCUE-ArduBooster C6
+L C C6
 U 1 1 54D7FAD7
 P 6950 3650
 F 0 "C6" H 7000 3750 50  0000 L CNN
 F 1 "22p" H 7000 3550 50  0000 L CNN
-F 2 "ArduBooster_Library:CAP_SMALL" H 6988 3500 30  0001 C CNN
+F 2 "Capacitors_ThroughHole:C_Rect_L7_W2_P5" H 6988 3500 30  0001 C CNN
 F 3 "" H 6950 3650 60  0000 C CNN
 	1    6950 3650
@@
 $EndComp
 Wire Wire Line
-	7250 3800 7250 2950
-Wire Wire Line
-	7250 2950 7150 2950
-Wire Wire Line
-	7150 3650 7250 3650
+	7250 2950 7250 3800
+Wire Wire Line
+	7100 2950 7250 2950
+Wire Wire Line
+	7100 3650 7250 3650
 Connection ~ 7250 3650
 $Comp
@@
 $EndComp
 $Comp
-L C-RESCUE-ArduBooster C7
+L C C7
 U 1 1 54D7FCE4
 P 7500 4350
 F 0 "C7" H 7550 4450 50  0000 L CNN
 F 1 "1u" H 7550 4250 50  0000 L CNN
-F 2 "ArduBooster_Library:CAP_BIG" H 7538 4200 30  0001 C CNN
+F 2 "Capacitors_ThroughHole:C_Rect_L7_W4.5_P5" H 7538 4200 30  0001 C CNN
 F 3 "" H 7500 4350 60  0000 C CNN
 	1    7500 4350
@@
 $EndComp
 $Comp
-L R-RESCUE-ArduBooster R4
+L R R4
 U 1 1 54D7FD1C
 P 7500 3800
@@
 $EndComp
 Wire Wire Line
-	7500 4600 7500 4550
-Wire Wire Line
-	7500 4150 7500 4050
-Wire Wire Line
-	7500 3550 7500 3500
+	7500 4500 7500 4600
+Wire Wire Line
+	7500 3950 7500 4200
+Wire Wire Line
+	7500 3500 7500 3650
 Wire Wire Line
 	4600 4100 7500 4100
 Connection ~ 7500 4100
 $Comp
-L R-RESCUE-ArduBooster R2
+L R R2
 U 1 1 54D7FEF8
 P 5200 5500
@@
 $EndComp
 $Comp
-L R-RESCUE-ArduBooster R3
+L R R3
 U 1 1 54D7FF4D
 P 5200 5700
@@
 	4650 4950 4650 5700
 Wire Wire Line
-	4650 5700 4950 5700
+	4650 5700 5050 5700
 Wire Wire Line
 	4600 4850 4750 4850
@@
 	4750 4850 4750 5500
 Wire Wire Line
-	4750 5500 4950 5500
-Wire Wire Line
-	5650 5500 5450 5500
-Wire Wire Line
-	5650 5700 5450 5700
-$Comp
-L R-RESCUE-ArduBooster R5
+	4750 5500 5050 5500
+Wire Wire Line
+	5350 5500 5650 5500
+Wire Wire Line
+	5350 5700 5650 5700
+$Comp
+L R R5
 U 1 1 54D8030D
 P 5050 4750
@@
 $EndComp
 Wire Wire Line
-	5050 4500 5050 4450
+	5050 4450 5050 4600
 Connection ~ 5050 4450
 $Comp
@@
 $EndComp
 Wire Wire Line
-	5050 5200 5050 5000
+	5050 4900 5050 5200
 NoConn ~ 4600 4750
 NoConn ~ 4600 4650
@@
 NoConn ~ 4600 2650
 $Comp
-L R-RESCUE-ArduBooster R6
+L R R6
 U 1 1 54D809E7
 P 4900 2150
@@
 $EndComp
 $Comp
-L R-RESCUE-ArduBooster R7
+L R R7
 U 1 1 54D80AC6
 P 5100 2150
@@
 $EndComp
 Wire Wire Line
-	5450 3850 5100 3850
-Wire Wire Line
-	5100 3850 5100 2400
-Wire Wire Line
-	5450 4000 4900 4000
-Wire Wire Line
-	4900 4000 4900 2400
+	5100 3850 5450 3850
+Wire Wire Line
+	5100 2300 5100 3850
+Wire Wire Line
+	4900 4000 5450 4000
+Wire Wire Line
+	4900 2300 4900 4000
 Wire Wire Line
 	4600 3500 5100 3500
@@
 $EndComp
 Wire Wire Line
-	4900 1900 4900 1850
+	4900 1850 4900 2000
 Wire Wire Line
 	4900 1850 5100 1850
 Wire Wire Line
-	5100 1850 5100 1900
+	5100 1850 5100 2000
 Wire Wire Line
 	5000 1700 5000 1850
@@
 	4600 2950 5200 2950
 $Comp
-L R-RESCUE-ArduBooster R8
+L R R8
 U 1 1 54D81783
 P 6500 1650
@@
 $EndComp
 $Comp
-L R-RESCUE-ArduBooster R9
+L R R9
 U 1 1 54D8179E
 P 6500 1900
@@
 $EndComp
 $Comp
-L C-RESCUE-ArduBooster C8
+L C C8
 U 1 1 54D8180B
 P 6900 2200
 F 0 "C8" H 6950 2300 50  0000 L CNN
 F 1 "100n" H 6950 2100 50  0000 L CNN
-F 2 "ArduBooster_Library:CAP_MID" H 6938 2050 30  0001 C CNN
+F 2 "Capacitors_ThroughHole:C_Rect_L7_W2.5_P5" H 6938 2050 30  0001 C CNN
 F 3 "" H 6900 2200 60  0000 C CNN
 	1    6900 2200
@@
 $EndComp
 $Comp
-L C-RESCUE-ArduBooster C9
+L C C9
 U 1 1 54D81846
 P 7300 2200
 F 0 "C9" H 7350 2300 50  0000 L CNN
 F 1 "100n" H 7350 2100 50  0000 L CNN
-F 2 "ArduBooster_Library:CAP_MID" H 7338 2050 30  0001 C CNN
+F 2 "Capacitors_ThroughHole:C_Rect_L7_W2.5_P5" H 7338 2050 30  0001 C CNN
 F 3 "" H 7300 2200 60  0000 C CNN
 	1    7300 2200
@@
 $EndComp
 Wire Wire Line
-	6750 1900 7650 1900
-Wire Wire Line
-	6900 1900 6900 2000
-Wire Wire Line
-	6750 1650 7650 1650
+	6650 1900 7650 1900
+Wire Wire Line
+	6900 1900 6900 2050
+Wire Wire Line
+	6650 1650 7650 1650
 $Comp
 L GNDREF #PWR020
@@
 $EndComp
 Wire Wire Line
-	6900 2500 7300 2500
-Wire Wire Line
-	6900 2500 6900 2400
+	7300 2500 6900 2500
+Wire Wire Line
+	6900 2500 6900 2350
 Wire Wire Line
 	7100 2600 7100 2500
 Connection ~ 7100 2500
 Wire Wire Line
-	7300 2500 7300 2400
-Wire Wire Line
-	7300 1650 7300 2000
+	7300 2350 7300 2500
+Wire Wire Line
+	7300 1650 7300 2050
 Wire Wire Line
 	4600 2850 6100 2850
@@
 	6100 2850 6100 1900
 Wire Wire Line
-	6100 1900 6250 1900
+	6100 1900 6350 1900
 Wire Wire Line
 	4600 2750 6000 2750
@@
 	6000 2750 6000 1650
 Wire Wire Line
-	6000 1650 6250 1650
+	6000 1650 6350 1650
 Connection ~ 6900 1900
 Connection ~ 7300 1650
@@
 Text HLabel 7650 1650 2    60   Output ~ 0
 CH0_ARDUINO_SIG
+$Comp
+L +5V #PWR021
+U 1 1 57BC9586
+P 1650 3400
+F 0 "#PWR021" H 1650 3250 60  0001 C CNN
+F 1 "+5V" H 1650 3540 60  0000 C CNN
+F 2 "" H 1650 3400 60  0000 C CNN
+F 3 "" H 1650 3400 60  0000 C CNN
+	1    1650 3400
+	1    0    0    -1
+$EndComp
+$Comp
+L GNDREF #PWR022
+U 1 1 57BC95BE
+P 1650 3800
+F 0 "#PWR022" H 1650 3550 60  0001 C CNN
+F 1 "GNDREF" H 1650 3650 60  0000 C CNN
+F 2 "" H 1650 3800 60  0000 C CNN
+F 3 "" H 1650 3800 60  0000 C CNN
+	1    1650 3800
+	1    0    0    -1
+$EndComp
+$Comp
+L C C10
+U 1 1 57BC9625
+P 1650 3600
+AR Path="/54D7EFEF/57BC9625" Ref="C10"  Part="1"
+AR Path="/54D7C565/57BC9625" Ref="C?"  Part="1"
+F 0 "C10" H 1675 3700 50  0000 L CNN
+F 1 "100nF" H 1675 3500 50  0000 L CNN
+F 2 "Capacitors_ThroughHole:C_Rect_L7_W2.5_P5" H 1688 3450 50  0001 C CNN
+F 3 "" H 1650 3600 50  0000 C CNN
+	1    1650 3600
+	1    0    0    -1
+$EndComp
+Wire Wire Line
+	1650 3800 1650 3750
+Wire Wire Line
+	1650 3450 1650 3400
 $EndSCHEMATC

Commit message: New connectors connection. Labels corrections (direction).
Connections:
- net RESET: now reaches C7.1, IC1.1 ((PCINT14/~RESET~)PC6), R4.2
- net MISO: now reaches IC1.18 ((PCINT4/MISO)PB4)
- net SCK: now reaches IC1.19 ((PCINT5/SCK)PB5)
- net RX: now reaches IC1.2 ((PCINT16/RXD)PD0)
- net TX: now reaches IC1.3 ((PCINT17/TXD)PD1)
- net OUTPUT_SELECTION renamed MOSI
- no-connect marks 13 -> 9
Changed lines of the file:
@@
 $EndComp
 $Comp
-L GNDREF #PWR013
+L GNDREF #PWR015
 U 1 1 54D7F6B2
 P 2550 5150
-F 0 "#PWR013" H 2550 4900 60  0001 C CNN
+F 0 "#PWR015" H 2550 4900 60  0001 C CNN
 F 1 "GNDREF" H 2550 5000 60  0000 C CNN
 F 2 "" H 2550 5150 60  0000 C CNN
@@
 NoConn ~ 2700 3250
 $Comp
-L +5V #PWR014
+L +5V #PWR016
 U 1 1 54D7F7B3
 P 2550 2300
-F 0 "#PWR014" H 2550 2150 60  0001 C CNN
+F 0 "#PWR016" H 2550 2150 60  0001 C CNN
 F 1 "+5V" H 2550 2440 60  0000 C CNN
 F 2 "" H 2550 2300 60  0000 C CNN
@@
 	0    -1   -1   0
 $EndComp
-Wire Wire Line
-	2550 5150 2550 4850
-Wire Wire Line
-	2550 4850 2700 4850
-Wire Wire Line
-	2700 4950 2550 4950
-Connection ~ 2550 4950
-Wire Wire Line
-	2550 2300 2550 2950
-Wire Wire Line
-	2550 2650 2700 2650
-Wire Wire Line
-	2550 2950 2700 2950
-Connection ~ 2550 2650
-Wire Wire Line
-	4600 3350 6250 3350
-Wire Wire Line
-	6250 3350 6250 3650
-Wire Wire Line
-	6250 3650 6800 3650
-Wire Wire Line
-	6500 3450 6500 3650
-Wire Wire Line
-	4600 3250 6250 3250
-Wire Wire Line
-	6250 3250 6250 2950
-Wire Wire Line
-	6250 2950 6800 2950
-Wire Wire Line
-	6500 2950 6500 3150
 $Comp
 L C C5
@@
 	0    1    1    0
 $EndComp
-Connection ~ 6500 3650
-Connection ~ 6500 2950
-$Comp
-L GNDREF #PWR015
+$Comp
+L GNDREF #PWR017
 U 1 1 54D7FB6B
 P 7250 3800
-F 0 "#PWR015" H 7250 3550 60  0001 C CNN
+F 0 "#PWR017" H 7250 3550 60  0001 C CNN
 F 1 "GNDREF" H 7250 3650 60  0000 C CNN
 F 2 "" H 7250 3800 60  0000 C CNN
@@
 	1    0    0    -1
 $EndComp
-Wire Wire Line
-	7250 2950 7250 3800
-Wire Wire Line
-	7100 2950 7250 2950
-Wire Wire Line
-	7100 3650 7250 3650
-Connection ~ 7250 3650
-$Comp
-L GNDREF #PWR016
+$Comp
+L GNDREF #PWR018
 U 1 1 54D7FCBC
 P 7500 4600
-F 0 "#PWR016" H 7500 4350 60  0001 C CNN
+F 0 "#PWR018" H 7500 4350 60  0001 C CNN
 F 1 "GNDREF" H 7500 4450 60  0000 C CNN
 F 2 "" H 7500 4600 60  0000 C CNN
@@
 $EndComp
 $Comp
-L +5V #PWR017
+L +5V #PWR019
 U 1 1 54D7FCD0
 P 7500 3500
-F 0 "#PWR017" H 7500 3350 60  0001 C CNN
+F 0 "#PWR019" H 7500 3350 60  0001 C CNN
 F 1 "+5V" H 7500 3640 60  0000 C CNN
 F 2 "" H 7500 3500 60  0000 C CNN
@@
 	1    0    0    -1
 $EndComp
-Wire Wire Line
-	7500 4500 7500 4600
-Wire Wire Line
-	7500 3950 7500 4200
-Wire Wire Line
-	7500 3500 7500 3650
-Wire Wire Line
-	4600 4100 7500 4100
-Connection ~ 7500 4100
 $Comp
 L R R2
@@
 	0    1    1    0
 $EndComp
-Wire Wire Line
-	4600 4950 4650 4950
-Wire Wire Line
-	4650 4950 4650 5700
-Wire Wire Line
-	4650 5700 5050 5700
-Wire Wire Line
-	4600 4850 4750 4850
-Wire Wire Line
-	4750 4850 4750 5500
-Wire Wire Line
-	4750 5500 5050 5500
-Wire Wire Line
-	5350 5500 5650 5500
-Wire Wire Line
-	5350 5700 5650 5700
 $Comp
 L R R5
@@
 	1    0    0    -1
 $EndComp
-Wire Wire Line
-	5050 4450 5050 4600
-Connection ~ 5050 4450
-$Comp
-L GNDREF #PWR018
+$Comp
+L GNDREF #PWR020
 U 1 1 54D8038E
 P 5050 5200
-F 0 "#PWR018" H 5050 4950 60  0001 C CNN
+F 0 "#PWR020" H 5050 4950 60  0001 C CNN
 F 1 "GNDREF" H 5050 5050 60  0000 C CNN
 F 2 "" H 5050 5200 60  0000 C CNN
@@
 	1    0    0    -1
 $EndComp
-Wire Wire Line
-	5050 4900 5050 5200
 NoConn ~ 4600 4750
 NoConn ~ 4600 4650
 NoConn ~ 4600 4550
-NoConn ~ 4600 4350
-NoConn ~ 4600 4250
 NoConn ~ 4600 3700
 NoConn ~ 4600 3800
 NoConn ~ 4600 3900
 NoConn ~ 4600 4000
-NoConn ~ 4600 3050
-NoConn ~ 4600 3150
 NoConn ~ 4600 2650
 $Comp
@@
 	1    0    0    -1
 $EndComp
-Wire Wire Line
-	5100 3850 5450 3850
-Wire Wire Line
-	5100 2300 5100 3850
-Wire Wire Line
-	4900 4000 5450 4000
-Wire Wire Line
-	4900 2300 4900 4000
-Wire Wire Line
-	4600 3500 5100 3500
-Connection ~ 5100 3500
-Wire Wire Line
-	4600 3600 4900 3600
-Connection ~ 4900 3600
-$Comp
-L +5V #PWR019
+$Comp
+L +5V #PWR021
 U 1 1 54D80C81
 P 5000 1700
-F 0 "#PWR019" H 5000 1550 60  0001 C CNN
+F 0 "#PWR021" H 5000 1550 60  0001 C CNN
 F 1 "+5V" H 5000 1840 60  0000 C CNN
 F 2 "" H 5000 1700 60  0000 C CNN
@@
 	1    0    0    -1
 $EndComp
-Wire Wire Line
-	4900 1850 4900 2000
-Wire Wire Line
-	4900 1850 5100 1850
-Wire Wire Line
-	5100 1850 5100 2000
-Wire Wire Line
-	5000 1700 5000 1850
-Connection ~ 5000 1850
-Wire Wire Line
-	4600 2950 5200 2950
 $Comp
 L R R8
@@
 	1    0    0    -1
 $EndComp
-Wire Wire Line
-	6650 1900 7650 1900
-Wire Wire Line
-	6900 1900 6900 2050
-Wire Wire Line
-	6650 1650 7650 1650
-$Comp
-L GNDREF #PWR020
+$Comp
+L GNDREF #PWR022
 U 1 1 54D8194E
 P 7100 2600
-F 0 "#PWR020" H 7100 2350 60  0001 C CNN
+F 0 "#PWR022" H 7100 2350 60  0001 C CNN
 F 1 "GNDREF" H 7100 2450 60  0000 C CNN
 F 2 "" H 7100 2600 60  0000 C CNN
@@
 	1    0    0    -1
 $EndComp
-Wire Wire Line
-	7300 2500 6900 2500
-Wire Wire Line
-	6900 2500 6900 2350
-Wire Wire Line
-	7100 2600 7100 2500
-Connection ~ 7100 2500
-Wire Wire Line
-	7300 2350 7300 2500
-Wire Wire Line
-	7300 1650 7300 2050
-Wire Wire Line
-	4600 2850 6100 2850
-Wire Wire Line
-	6100 2850 6100 1900
-Wire Wire Line
-	6100 1900 6350 1900
-Wire Wire Line
-	4600 2750 6000 2750
-Wire Wire Line
-	6000 2750 6000 1650
-Wire Wire Line
-	6000 1650 6350 1650
-Connection ~ 6900 1900
-Connection ~ 7300 1650
-Wire Wire Line
-	4600 4450 5250 4450
-Text HLabel 5250 4450 2    60   Output ~ 0
+Text HLabel 5250 4450 2    60   Input ~ 0
 SWITCH
-Text HLabel 5450 4000 2    60   Output ~ 0
+Text HLabel 5450 4000 2    60   Input ~ 0
 CH1_PEDAL_SIG
-Text HLabel 5450 3850 2    60   Output ~ 0
+Text HLabel 5450 3850 2    60   Input ~ 0
 CH0_PEDAL_SIG
-Text HLabel 5650 5500 2    60   Input ~ 0
+Text HLabel 5650 5500 2    60   Output ~ 0
 LED1
-Text HLabel 5650 5700 2    60   Input ~ 0
+Text HLabel 5650 5700 2    60   Output ~ 0
 LED2
 Text HLabel 5200 2950 2    60   Output ~ 0
@@
 CH0_ARDUINO_SIG
 $Comp
-L +5V #PWR021
+L +5V #PWR023
 U 1 1 57BC9586
 P 1650 3400
-F 0 "#PWR021" H 1650 3250 60  0001 C CNN
+F 0 "#PWR023" H 1650 3250 60  0001 C CNN
 F 1 "+5V" H 1650 3540 60  0000 C CNN
 F 2 "" H 1650 3400 60  0000 C CNN
@@
 $EndComp
 $Comp
-L GNDREF #PWR022
+L GNDREF #PWR024
 U 1 1 57BC95BE
 P 1650 3800
-F 0 "#PWR022" H 1650 3550 60  0001 C CNN
+F 0 "#PWR024" H 1650 3550 60  0001 C CNN
 F 1 "GNDREF" H 1650 3650 60  0000 C CNN
 F 2 "" H 1650 3800 60  0000 C CNN
@@
 	1    0    0    -1
 $EndComp
+Text HLabel 4200 2000 0    60   Input ~ 0
+SCK
+Text HLabel 4200 2100 0    60   Input ~ 0
+MISO
+Text HLabel 4200 2200 0    60   Output ~ 0
+MOSI
+Wire Wire Line
+	2550 5150 2550 4850
+Wire Wire Line
+	2550 4850 2700 4850
+Wire Wire Line
+	2700 4950 2550 4950
+Connection ~ 2550 4950
+Wire Wire Line
+	2550 2300 2550 2950
+Wire Wire Line
+	2550 2650 2700 2650
+Wire Wire Line
+	2550 2950 2700 2950
+Connection ~ 2550 2650
+Wire Wire Line
+	4600 3350 6250 3350
+Wire Wire Line
+	6250 3350 6250 3650
+Wire Wire Line
+	6250 3650 6800 3650
+Wire Wire Line
+	6500 3450 6500 3650
+Wire Wire Line
+	4600 3250 6250 3250
+Wire Wire Line
+	6250 3250 6250 2950
+Wire Wire Line
+	6250 2950 6800 2950
+Wire Wire Line
+	6500 2950 6500 3150
+Connection ~ 6500 3650
+Connection ~ 6500 2950
+Wire Wire Line
+	7250 2950 7250 3800
+Wire Wire Line
+	7100 2950 7250 2950
+Wire Wire Line
+	7100 3650 7250 3650
+Connection ~ 7250 3650
+Wire Wire Line
+	7500 4500 7500 4600
+Wire Wire Line
+	7500 3950 7500 4200
+Wire Wire Line
+	7500 3500 7500 3650
+Wire Wire Line
+	4600 4100 7500 4100
+Connection ~ 7500 4100
+Wire Wire Line
+	4600 4950 4650 4950
+Wire Wire Line
+	4650 4950 4650 5700
+Wire Wire Line
+	4650 5700 5050 5700
+Wire Wire Line
+	4600 4850 4750 4850
+Wire Wire Line
+	4750 4850 4750 5500
+Wire Wire Line
+	4750 5500 5050 5500
+Wire Wire Line
+	5350 5500 5650 5500
+Wire Wire Line
+	5350 5700 5650 5700
+Wire Wire Line
+	5050 4450 5050 4600
+Connection ~ 5050 4450
+Wire Wire Line
+	5050 4900 5050 5200
+Wire Wire Line
+	5100 3850 5450 3850
+Wire Wire Line
+	5100 2300 5100 3850
+Wire Wire Line
+	4900 4000 5450 4000
+Wire Wire Line
+	4900 2300 4900 4000
+Wire Wire Line
+	4600 3500 5100 3500
+Connection ~ 5100 3500
+Wire Wire Line
+	4600 3600 4900 3600
+Connection ~ 4900 3600
+Wire Wire Line
+	4900 1850 4900 2000
+Wire Wire Line
+	4900 1850 5100 1850
+Wire Wire Line
+	5100 1850 5100 2000
+Wire Wire Line
+	5000 1700 5000 1850
+Connection ~ 5000 1850
+Wire Wire Line
+	4600 2950 5200 2950
+Wire Wire Line
+	6650 1900 7650 1900
+Wire Wire Line
+	6900 1900 6900 2050
+Wire Wire Line
+	6650 1650 7650 1650
+Wire Wire Line
+	7300 2500 6900 2500
+Wire Wire Line
+	6900 2500 6900 2350
+Wire Wire Line
+	7100 2600 7100 2500
+Connection ~ 7100 2500
+Wire Wire Line
+	7300 2350 7300 2500
+Wire Wire Line
+	7300 1650 7300 2050
+Wire Wire Line
+	4600 2850 6100 2850
+Wire Wire Line
+	6100 2850 6100 1900
+Wire Wire Line
+	6100 1900 6350 1900
+Wire Wire Line
+	4600 2750 6000 2750
+Wire Wire Line
+	6000 2750 6000 1650
+Wire Wire Line
+	6000 1650 6350 1650
+Connection ~ 6900 1900
+Connection ~ 7300 1650
+Wire Wire Line
+	4600 4450 5250 4450
 Wire Wire Line
 	1650 3800 1650 3750
 Wire Wire Line
 	1650 3450 1650 3400
+Wire Wire Line
+	4200 2200 4650 2200
+Wire Wire Line
+	4650 2200 4650 2950
+Connection ~ 4650 2950
+Wire Wire Line
+	4200 2100 4700 2100
+Wire Wire Line
+	4700 2100 4700 3050
+Wire Wire Line
+	4700 3050 4600 3050
+Wire Wire Line
+	4200 2000 4750 2000
+Wire Wire Line
+	4750 2000 4750 3150
+Wire Wire Line
+	4750 3150 4600 3150
+Text HLabel 6500 4300 3    60   Input ~ 0
+RESET
+Wire Wire Line
+	6500 4300 6500 4100
+Connection ~ 6500 4100
+Text HLabel 4900 4250 2    60   Input ~ 0
+RX
+Text HLabel 4900 4350 2    60   Output ~ 0
+TX
+Wire Wire Line
+	4900 4250 4600 4250
+Wire Wire Line
+	4600 4350 4900 4350
 $EndSCHEMATC

Commit message: Correct DIP sockets footprints.
Parts:
- IC1: footprint Sockets_DIP:DIP-28__300 -> Housings_DIP:DIP-28_W7.62mm_LongPads
Changed lines of the file:
@@
 F 0 "IC1" H 2850 5000 40  0000 L BNN
 F 1 "ATMEGA328-P" H 4000 2350 40  0000 L BNN
-F 2 "Sockets_DIP:DIP-28__300" H 3600 3750 30  0001 C CIN
+F 2 "Housings_DIP:DIP-28_W7.62mm_LongPads" H 3600 3750 30  0001 C CIN
 F 3 "" H 3600 3750 60  0000 C CNN
 	1    3600 3750
