File: PCB/Doubler_Inverter.sch (KiCad schematic (older format))
At the start: 7 parts, among them U1 ICL7660

Commit message: Libraries and footprints adjustments. New connectors (4 pins main, 2 pins debug and 6 pins isp). New source input cap.
Parts:
- C1, C2, C3, C4: footprint ArduBooster_Library:CAP_BIG -> Capacitors_ThroughHole:C_Rect_L7_W4.5_P5; symbol C-RESCUE-ArduBooster -> C
- D1, D2: footprint ArduBooster_Library:DIODE -> Discret:D3; symbol DIODE -> D
Connections:
- net +5V: now also D1.2 (A); no longer D1.1 (A)
- net +9V: now also D2.1 (K); no longer D2.2 (K)
- new net: C2.1, D1.1 (K), D2.2 (A)
Changed lines of the file:
@@
 EESchema Schematic File Version 2
-LIBS:ArduBooster-rescue
 LIBS:power
 LIBS:device
@@
 Rev "1.0"
 Comp ""
-Comment1 "Input: 0V/5V"
-Comment2 "Output: -5V/9V"
-Comment3 ""
+Comment1 "Output: -5V/9V"
+Comment2 "Input: 0V/5V"
+Comment3 "Doubler/Inverter - Source to OpAmp"
 Comment4 ""
 $EndDescr
@@
 $EndComp
 $Comp
-L C-RESCUE-ArduBooster C1
+L C C1
 U 1 1 54D7C587
 P 3800 3550
 F 0 "C1" H 3850 3650 50  0000 L CNN
 F 1 "1u" H 3850 3450 50  0000 L CNN
-F 2 "ArduBooster_Library:CAP_BIG" H 3838 3400 30  0001 C CNN
+F 2 "Capacitors_ThroughHole:C_Rect_L7_W4.5_P5" H 3838 3400 30  0001 C CNN
 F 3 "" H 3800 3550 60  0000 C CNN
 	1    3800 3550
@@
 $EndComp
 $Comp
-L C-RESCUE-ArduBooster C2
+L C C2
 U 1 1 54D7C5F6
 P 5650 4550
 F 0 "C2" H 5700 4650 50  0000 L CNN
 F 1 "1u" H 5700 4450 50  0000 L CNN
-F 2 "ArduBooster_Library:CAP_BIG" H 5688 4400 30  0001 C CNN
+F 2 "Capacitors_ThroughHole:C_Rect_L7_W4.5_P5" H 5688 4400 30  0001 C CNN
 F 3 "" H 5650 4550 60  0000 C CNN
 	1    5650 4550
@@
 $EndComp
 $Comp
-L C-RESCUE-ArduBooster C3
+L C C3
 U 1 1 54D7C60F
 P 7200 4950
 F 0 "C3" H 7250 5050 50  0000 L CNN
 F 1 "1u" H 7250 4850 50  0000 L CNN
-F 2 "ArduBooster_Library:CAP_BIG" H 7238 4800 30  0001 C CNN
+F 2 "Capacitors_ThroughHole:C_Rect_L7_W4.5_P5" H 7238 4800 30  0001 C CNN
 F 3 "" H 7200 4950 60  0000 C CNN
 	1    7200 4950
@@
 $EndComp
 $Comp
-L C-RESCUE-ArduBooster C4
+L C C4
 U 1 1 54D7C66C
 P 7600 4950
 F 0 "C4" H 7650 5050 50  0000 L CNN
 F 1 "1u" H 7650 4850 50  0000 L CNN
-F 2 "ArduBooster_Library:CAP_BIG" H 7638 4800 30  0001 C CNN
+F 2 "Capacitors_ThroughHole:C_Rect_L7_W4.5_P5" H 7638 4800 30  0001 C CNN
 F 3 "" H 7600 4950 60  0000 C CNN
 	1    7600 4950
@@
 $EndComp
 $Comp
-L DIODE D1
+L D D1
 U 1 1 54D7C6AB
 P 6400 4150
 F 0 "D1" H 6400 4250 50  0000 C CNN
 F 1 "1n4007" H 6400 4050 50  0000 C CNN
-F 2 "ArduBooster_Library:DIODE" H 6400 4150 60  0001 C CNN
+F 2 "Discret:D3" H 6400 4150 60  0001 C CNN
 F 3 "" H 6400 4150 60  0000 C CNN
 	1    6400 4150
-	0    1    1    0
-$EndComp
-$Comp
-L DIODE D2
+	0    -1   -1   0
+$EndComp
+$Comp
+L D D2
 U 1 1 54D7C6F0
 P 6800 4550
 F 0 "D2" H 6800 4650 50  0000 C CNN
 F 1 "1n4007" H 6800 4450 50  0000 C CNN
-F 2 "ArduBooster_Library:DIODE" H 6800 4550 60  0001 C CNN
+F 2 "Discret:D3" H 6800 4550 60  0001 C CNN
 F 3 "" H 6800 4550 60  0000 C CNN
 	1    6800 4550
-	1    0    0    -1
+	-1   0    0    1
 $EndComp
 NoConn ~ 4400 3850
@@
 	4000 3250 3800 3250
 Wire Wire Line
-	3800 3250 3800 3350
+	3800 3250 3800 3400
 Wire Wire Line
 	4400 3650 4000 3650
@@
 	4000 3850 3800 3850
 Wire Wire Line
-	3800 3850 3800 3750
-Wire Wire Line
-	5450 4550 4250 4550
+	3800 3850 3800 3700
+Wire Wire Line
+	4250 4550 5500 4550
 Wire Wire Line
 	4250 4550 4250 3450
 Connection ~ 4250 3450
 Wire Wire Line
-	5850 4550 6600 4550
-Wire Wire Line
-	6400 4350 6400 4550
+	5800 4550 6650 4550
+Wire Wire Line
+	6400 4300 6400 4550
 Connection ~ 6400 4550
 Wire Wire Line
-	6400 3950 6400 2950
+	6400 2950 6400 4000
 Wire Wire Line
 	6400 2950 5200 2950
@@
 	5200 2800 5200 3050
 Wire Wire Line
-	7000 4550 7900 4550
-Wire Wire Line
-	7200 4550 7200 4750
-Wire Wire Line
-	7600 4750 7600 3550
+	6950 4550 7900 4550
+Wire Wire Line
+	7200 4550 7200 4800
+Wire Wire Line
+	7600 3550 7600 4800
 Wire Wire Line
 	6100 3550 7900 3550
@@
 Connection ~ 7200 4550
 Wire Wire Line
-	7600 5150 7600 5250
+	7600 5100 7600 5250
 Wire Wire Line
 	7600 5250 7200 5250
 Wire Wire Line
-	7200 5250 7200 5150
+	7200 5250 7200 5100
 Wire Wire Line
 	7400 5350 7400 5250

Commit message: New connectors connection. Labels corrections (direction).
Changed lines of the file:
@@
 NoConn ~ 6100 3850
 $Comp
-L GNDREF #PWR07
+L GNDREF #PWR09
 U 1 1 54D7CA46
 P 7400 5350
-F 0 "#PWR07" H 7400 5100 60  0001 C CNN
+F 0 "#PWR09" H 7400 5100 60  0001 C CNN
 F 1 "GNDREF" H 7400 5200 60  0000 C CNN
 F 2 "" H 7400 5350 60  0000 C CNN
@@
 $EndComp
 $Comp
-L GNDREF #PWR08
+L GNDREF #PWR010
 U 1 1 54D7CAA6
 P 5200 4700
-F 0 "#PWR08" H 5200 4450 60  0001 C CNN
+F 0 "#PWR010" H 5200 4450 60  0001 C CNN
 F 1 "GNDREF" H 5200 4550 60  0000 C CNN
 F 2 "" H 5200 4700 60  0000 C CNN
@@
 $EndComp
 $Comp
-L +5V #PWR09
+L +5V #PWR011
 U 1 1 54D7CB10
 P 5200 2800
-F 0 "#PWR09" H 5200 2650 60  0001 C CNN
+F 0 "#PWR011" H 5200 2650 60  0001 C CNN
 F 1 "+5V" H 5200 2940 60  0000 C CNN
 F 2 "" H 5200 2800 60  0000 C CNN
@@
 Connection ~ 5200 2950
 $Comp
-L PWR_FLAG #FLG010
+L PWR_FLAG #FLG012
 U 1 1 54D7D3CB
 P 7750 4350
-F 0 "#FLG010" H 7750 4445 30  0001 C CNN
+F 0 "#FLG012" H 7750 4445 30  0001 C CNN
 F 1 "PWR_FLAG" H 7750 4530 30  0000 C CNN
 F 2 "" H 7750 4350 60  0000 C CNN
@@
 	7750 4350 7750 4550
 Connection ~ 7750 4550
-Text HLabel 7900 3550 2    60   Output ~ 0
+Text HLabel 7900 3550 2    60   Input ~ 0
 -5V
 Text HLabel 7900 4550 2    60   Output ~ 0

Commit message: Correct DIP sockets footprints.
Parts:
- U1: footprint Sockets_DIP:DIP-8__300 -> Housings_DIP:DIP-8_W7.62mm_LongPads
Changed lines of the file:
@@
 F 0 "U1" H 5450 4100 70  0000 L CNN
 F 1 "ICL7660" H 5300 3250 70  0000 L CNN
-F 2 "Sockets_DIP:DIP-8__300" H 5250 3700 60  0001 C CNN
+F 2 "Housings_DIP:DIP-8_W7.62mm_LongPads" H 5250 3700 60  0001 C CNN
 F 3 "" H 5250 3700 60  0000 C CNN
 	1    5250 3700

Commit message: Last commit before Mux/Demux removel. Single layer PCB incompete (3 wires). Add ADC input filter.
Parts:
- C1, C2, C3, C4: footprint Capacitors_ThroughHole:C_Rect_L7_W4.5_P5 -> Capacitors_THT:C_Rect_L7.0mm_W4.5mm_P5.00mm
- D1, D2: footprint Discret:D3 -> Diodes_THT:D_A-405_P2.54mm_Vertical_AnodeUp
Changed lines of the file:
@@
 Rev "1.0"
 Comp ""
-Comment1 "Output: -5V/9V"
-Comment2 "Input: 0V/5V"
-Comment3 "Doubler/Inverter - Source to OpAmp"
-Comment4 ""
+Comment1 "Used to ensure that OpAmp output will cover all  possible voltages (0V to 5V)"
+Comment2 "Output: -5V/9V"
+Comment3 "Input: 0V/5V"
+Comment4 "Doubler/Inverter - Power source to OpAmp"
 $EndDescr
 $Comp
@@
 F 0 "C1" H 3850 3650 50  0000 L CNN
 F 1 "1u" H 3850 3450 50  0000 L CNN
-F 2 "Capacitors_ThroughHole:C_Rect_L7_W4.5_P5" H 3838 3400 30  0001 C CNN
+F 2 "Capacitors_THT:C_Rect_L7.0mm_W4.5mm_P5.00mm" H 3838 3400 30  0001 C CNN
 F 3 "" H 3800 3550 60  0000 C CNN
 	1    3800 3550
@@
 F 0 "C2" H 5700 4650 50  0000 L CNN
 F 1 "1u" H 5700 4450 50  0000 L CNN
-F 2 "Capacitors_ThroughHole:C_Rect_L7_W4.5_P5" H 5688 4400 30  0001 C CNN
+F 2 "Capacitors_THT:C_Rect_L7.0mm_W4.5mm_P5.00mm" H 5688 4400 30  0001 C CNN
 F 3 "" H 5650 4550 60  0000 C CNN
 	1    5650 4550
@@
 F 0 "C3" H 7250 5050 50  0000 L CNN
 F 1 "1u" H 7250 4850 50  0000 L CNN
-F 2 "Capacitors_ThroughHole:C_Rect_L7_W4.5_P5" H 7238 4800 30  0001 C CNN
+F 2 "Capacitors_THT:C_Rect_L7.0mm_W4.5mm_P5.00mm" H 7238 4800 30  0001 C CNN
 F 3 "" H 7200 4950 60  0000 C CNN
 	1    7200 4950
@@
 F 0 "C4" H 7650 5050 50  0000 L CNN
 F 1 "1u" H 7650 4850 50  0000 L CNN
-F 2 "Capacitors_ThroughHole:C_Rect_L7_W4.5_P5" H 7638 4800 30  0001 C CNN
+F 2 "Capacitors_THT:C_Rect_L7.0mm_W4.5mm_P5.00mm" H 7638 4800 30  0001 C CNN
 F 3 "" H 7600 4950 60  0000 C CNN
 	1    7600 4950
@@
 F 0 "D1" H 6400 4250 50  0000 C CNN
 F 1 "1n4007" H 6400 4050 50  0000 C CNN
-F 2 "Discret:D3" H 6400 4150 60  0001 C CNN
+F 2 "Diodes_THT:D_A-405_P2.54mm_Vertical_AnodeUp" H 6400 4150 60  0001 C CNN
 F 3 "" H 6400 4150 60  0000 C CNN
 	1    6400 4150
@@
 F 0 "D2" H 6800 4650 50  0000 C CNN
 F 1 "1n4007" H 6800 4450 50  0000 C CNN
-F 2 "Discret:D3" H 6800 4550 60  0001 C CNN
+F 2 "Diodes_THT:D_A-405_P2.54mm_Vertical_AnodeUp" H 6800 4550 60  0001 C CNN
 F 3 "" H 6800 4550 60  0000 C CNN
 	1    6800 4550
